Commit message: Simplify URDF

File: test/urdf/chassis.xacro (robot description, xacro)
@@ -2,5 +2,4 @@
 <robot xmlns:xacro="http://www.ros.org/wiki/xacro" name="chassis">
   <!-- Base Properties -->
-  <xacro:property name="mass_base" value="340" />
   <xacro:property name="base_x_size" value="1.66000" />
   <xacro:property name="base_y_size" value="0.60000" />
@@ -12,24 +11,16 @@
     <link name="base_link">
       <visual>
-        <origin xyz="0 0 0" rpy="0 0 0" />
         <geometry>
-          <box size="${base_x_size} ${base_y_size} ${base_z_size}"/>
+          <box size="${base_x_size} ${base_y_size} ${base_z_size}" />
         </geometry>
         <material name="grey">
-          <color rgba="0.6 0.6 0.6 1"/>
+          <color rgba="0.6 0.6 0.6 1" />
         </material>
       </visual>
       <collision>
         <geometry>
-          <box size="${base_x_size} ${base_y_size} ${base_z_size}"/>
+          <box size="${base_x_size} ${base_y_size} ${base_z_size}" />
         </geometry>
       </collision>
-      <inertial>
-        <mass value="340" />
-        <origin xyz="0 0 0" />
-        <inertia ixx="${mass_base/12.0 * (base_y_size*base_y_size + base_z_size*base_z_size)}" ixy="0" ixz="0"
-                 iyy="${mass_base/12.0 * (base_x_size*base_x_size + base_z_size*base_z_size)}" iyz="0"
-                 izz="${mass_base/12.0 * (base_y_size*base_y_size + base_x_size*base_x_size)}" />
-      </inertial>
     </link>
   </xacro:macro>

File: test/urdf/four_wheel_steering.urdf.xacro (robot description, xacro)
@@ -3,26 +3,22 @@
   <xacro:include filename="$(find urdf_geometry_parser)/test/urdf/chassis.xacro" />
   <xacro:include filename="$(find urdf_geometry_parser)/test/urdf/wheel_steered.xacro" />
-  <xacro:property name="M_PI" value="3.14159"/>
+  <xacro:property name="M_PI" value="3.14159" />
   <!-- Wheel Mounting Positions -->
   <xacro:property name="ground_clearance" value="0.19" />
   <xacro:property name="wheel_x_offset" value="0.0" />
   <xacro:property name="wheel_y_offset" value="0.05" />
-  <xacro:chassis/>
+  <xacro:chassis />
   <!-- Wheel macros -->
-  <xacro:wheel_steered wheel_prefix="front_left" parent_link="base_link" wheel_origin_y="${wheel_y_offset}" left_right="-1">
-    <origin xyz="${wheelbase/2+wheel_x_offset} ${track/2-wheel_y_offset} ${-base_z_size/2 + wheel_radius - ground_clearance}" rpy="0 0 0" />
+  <xacro:wheel_steered wheel_prefix="front_left" parent_link="base_link" left_right="-1">
+    <origin xyz="${wheelbase/2+wheel_x_offset} ${track/2} ${-base_z_size/2 + wheel_radius - ground_clearance}" rpy="0 0 0" />
   </xacro:wheel_steered>
-  <xacro:wheel_steered wheel_prefix="front_right" parent_link="base_link" wheel_origin_y="${-wheel_y_offset}" left_right="1">
-    <origin xyz="${wheelbase/2+wheel_x_offset} ${-track/2+wheel_y_offset} ${-base_z_size/2 + wheel_radius - ground_clearance}" rpy="0 0 0" />
+  <xacro:wheel_steered wheel_prefix="front_right" parent_link="base_link" left_right="1">
+    <origin xyz="${wheelbase/2+wheel_x_offset} ${-track/2} ${-base_z_size/2 + wheel_radius - ground_clearance}" rpy="0 0 0" />
   </xacro:wheel_steered>
-  <xacro:wheel_steered wheel_prefix="rear_left" parent_link="base_link" wheel_origin_y="${wheel_y_offset}" left_right="-1">
-    <origin xyz="${-wheelbase/2+wheel_x_offset} ${track/2-wheel_y_offset} ${-base_z_size/2 + wheel_radius - ground_clearance}" rpy="0 0 0" />
+  <xacro:wheel_steered wheel_prefix="rear_left" parent_link="base_link" left_right="-1">
+    <origin xyz="${-wheelbase/2+wheel_x_offset} ${track/2} ${-base_z_size/2 + wheel_radius - ground_clearance}" rpy="0 0 0" />
   </xacro:wheel_steered>
-  <xacro:wheel_steered wheel_prefix="rear_right" parent_link="base_link" wheel_origin_y="${-wheel_y_offset}" left_right="1">
-    <origin xyz="${-wheelbase/2+wheel_x_offset} ${-track/2+wheel_y_offset} ${-base_z_size/2 + wheel_radius - ground_clearance}" rpy="0 0 0" />
+  <xacro:wheel_steered wheel_prefix="rear_right" parent_link="base_link" left_right="1">
+    <origin xyz="${-wheelbase/2+wheel_x_offset} ${-track/2} ${-base_z_size/2 + wheel_radius - ground_clearance}" rpy="0 0 0" />
   </xacro:wheel_steered>
-  <!-- Gazebo plugin for ROS Control -->
-  <gazebo>
-    <plugin name="gazebo_ros_control" filename="libgazebo_ros_control.so"/>
-  </gazebo>
 </robot>

File: test/urdf/wheel.xacro (robot description, xacro)
@@ -6,43 +6,27 @@
   <xacro:property name="mass_wheel" value="5.0" />
   <xacro:macro name="wheel" params="wheel_prefix parent_link left_right *joint_origin">
-		<link name="${wheel_prefix}_wheel_link">
-			<inertial>
-        <mass value="${mass_wheel}" />
-        <origin xyz="0 0 0" rpy="${M_PI/2}  0 0" />
-        <inertia  ixx="${mass_wheel/4.0*(wheel_radius*wheel_radius+wheel_length*wheel_length/3.0)}" ixy="0" ixz="0"
-                  iyy="${mass_wheel*wheel_radius*wheel_radius/2.0}" iyz="0"
-                  izz="${mass_wheel/4.0*(wheel_radius*wheel_radius+wheel_length*wheel_length/3.0)}" />
-      </inertial>
-			<visual>
-        <origin xyz="0 0 0" rpy="${left_right * M_PI/2}  0 0" />
-				<geometry>
-          <cylinder length="${wheel_length}" radius="${wheel_radius}"/>
-				</geometry>
+    <link name="${wheel_prefix}_wheel_link">
+      <visual>
+        <origin xyz="0 0 0" rpy="${left_right * M_PI/2} 0 0" />
+        <geometry>
+          <cylinder length="${wheel_length}" radius="${wheel_radius}" />
+        </geometry>
         <material name="black">
-          <color rgba="0 0 0 1"/>
+          <color rgba="0 0 0 1" />
         </material>
-			</visual>
-			<collision>
-				<origin xyz="0 0 0" rpy="${M_PI/2} 0 0" />
-				<geometry>
-					<cylinder length="${wheel_length}" radius="${wheel_radius}" />
-				</geometry>
-			</collision>
-		</link>
-		<joint name="${wheel_prefix}_wheel" type="continuous">
-      <parent link="${parent_link}"/>
-			<child link="${wheel_prefix}_wheel_link"/>
-      <xacro:insert_block name="joint_origin"/>
-			<axis xyz="0 1 0" rpy="0 0 0" />
-		</joint>
-		<transmission name="${wheel_prefix}_wheel_trans" type="SimpleTransmission">
-			<type>transmission_interface/SimpleTransmission</type>
-			<actuator name="${wheel_prefix}_wheel_motor">
-				<mechanicalReduction>1</mechanicalReduction>
-			</actuator>
-			<joint name="${wheel_prefix}_wheel">
-				<hardwareInterface>VelocityJointInterface</hardwareInterface>
-			</joint>
-		</transmission>
-	</xacro:macro>
+      </visual>
+      <collision>
+        <origin xyz="0 0 0" rpy="${M_PI/2} 0 0" />
+        <geometry>
+          <cylinder length="${wheel_length}" radius="${wheel_radius}" />
+        </geometry>
+      </collision>
+    </link>
+    <joint name="${wheel_prefix}_wheel" type="continuous">
+      <parent link="${parent_link}" />
+      <child link="${wheel_prefix}_wheel_link" />
+      <xacro:insert_block name="joint_origin" />
+      <axis xyz="0 1 0" />
+    </joint>
+  </xacro:macro>
 </robot>

File: test/urdf/wheel_steered.xacro (robot description, xacro)
@@ -1,46 +1,28 @@
 <?xml version="1.0"?>
 <robot xmlns:xacro="http://www.ros.org/wiki/xacro" name="wheel_steered">
-  <xacro:property name="steering_link_y" value="0.05" />
+  <xacro:property name="steering_link_y" value="${wheel_length + 0.1}" />
   <xacro:property name="steering_link_xz" value="0.1" />
-  <xacro:property name="steering_link_mass" value="5.0" />
   <xacro:include filename="$(find urdf_geometry_parser)/test/urdf/wheel.xacro" />
-  <xacro:macro name="wheel_steered" params="wheel_prefix parent_link wheel_origin_y left_right *joint_origin ">
+  <xacro:macro name="wheel_steered" params="wheel_prefix parent_link left_right *joint_origin ">
     <link name="${wheel_prefix}_steering">
       <visual>
-        <origin xyz="0 ${-wheel_origin_y} 0" rpy="0 0 0"/>
+        <origin xyz="0 0 0" rpy="0 0 0" />
         <geometry>
-          <box size="0.05 ${steering_link_y} 0.05"/>
+          <box size="${steering_link_xz} ${steering_link_y} ${steering_link_xz}" />
         </geometry>
         <material name="blue">
-          <color rgba="0.2 0.2 0.6 1"/>
+          <color rgba="0.2 0.2 0.6 1" />
         </material>
       </visual>
-      <inertial>
-        <mass value="${steering_link_mass}" />
-        <origin xyz="0 ${-wheel_origin_y} 0" />
-        <inertia  ixx="${steering_link_mass/12.0 * (steering_link_y*steering_link_y + steering_link_xz*steering_link_xz)}" ixy="0" ixz="0"
-                  iyy="${steering_link_mass/12.0 * (steering_link_xz*steering_link_xz + steering_link_xz*steering_link_xz)}" iyz="0"
-                  izz="${steering_link_mass/12.0 * (steering_link_y*steering_link_y + steering_link_xz*steering_link_xz)}" />
-      </inertial>
     </link>
     <joint name="${wheel_prefix}_steering_joint" type="revolute">
-      <limit lower="${-M_PI/6}" upper="${M_PI/6}" effort="1000.0" velocity="2.0"/>
-      <axis xyz="0 0 1"/>
-      <parent link="${parent_link}"/>
-      <child link="${wheel_prefix}_steering"/>
-      <xacro:insert_block name="joint_origin"/>
-      <dynamics damping="0.7"/>
+      <limit lower="${-M_PI/6}" upper="${M_PI/6}" effort="1000.0" velocity="2.0" />
+      <axis xyz="0 0 1" />
+      <parent link="${parent_link}" />
+      <child link="${wheel_prefix}_steering" />
+      <xacro:insert_block name="joint_origin" />
     </joint>
-    <transmission name="${wheel_prefix}_steering_trans" type="SimpleTransmission">
-      <type>transmission_interface/SimpleTransmission</type>
-      <actuator name="${wheel_prefix}_steering_motor">
-        <mechanicalReduction>1</mechanicalReduction>
-      </actuator>
-      <joint name="${wheel_prefix}_steering_joint">
-        <hardwareInterface>PositionJointInterface</hardwareInterface>
-      </joint>
-    </transmission>
     <xacro:wheel wheel_prefix="${wheel_prefix}" parent_link="${wheel_prefix}_steering" left_right="${left_right}">
-      <origin xyz="0 ${wheel_origin_y} 0" rpy="0 0 0" />
+      <origin xyz="0 0 0" rpy="0 0 0" />
     </xacro:wheel>
   </xacro:macro>
